Commit message: fix: decouple wall from robot URDF, clean .gitkeep, add runtime wave-maker switching
Remove the world/wall link+joint from simplified_v1_description's robot.xacro so
base_link is the sole URDF root (wall now lives only in MJCF physics and the
/rov/environment_markers RViz marker). Delete .gitkeep placeholders from
directories that now contain real sources. Replace the static wave_profile
launch-time binding in adhere_mujoco_hardware with runtime hot-swappable wave
switching: AdhereMujocoHardware always starts in Calm Water, exposes a
thread-safe setWaveMode()/activeInstance() pair driven by a new
/rov/wave_mode_cmd topic, and evaluates StationKeepingGustPlugin on a relative
wave clock (tau = t_sim - t_trigger) so gusts always replay from the moment the
wave-maker is switched on. Add an interactive wave_console_node terminal and
auto-spawn it from mujoco_sim.launch.py.

Co-Authored-By: Claude Sonnet 5 <noreply@anthropic.com>

File: src/descriptions/simplified_v1_description/urdf/simplified_v1.urdf.xacro (robot description, xacro)
@@ -1,5 +1,4 @@
 <?xml version="1.0"?>
 <robot name="simplified_v1" xmlns:xacro="http://www.ros.org/wiki/xacro">
-  <xacro:arg name="wave_profile" default="calm"/>
   <xacro:arg name="headless" default="false"/>
   <xacro:include filename="$(find simplified_v1_description)/xacro/robot.xacro"/>

File: src/descriptions/simplified_v1_description/xacro/robot.xacro (robot description, xacro)
@@ -3,8 +3,10 @@
   <!--
     Geometry mirrors mjcf/rov_wall.xml (and the read-only mujoco_mppi_ws reference) exactly:
-    wall at world X=0, rov_base chassis box 0.2x0.6x0.4 m, 4 spherical contact pads at
-    (-0.10, +/-0.25, +/-0.15) m, 8 thruster mount sites at X=0.0 with the same corner layout.
-    All non-base links are rigidly fixed; the only real DOF is the world->base_link floating
-    base, which is driven by AdhereMujocoHardware's free joint, not by any URDF joint.
+    rov_base chassis box 0.2x0.6x0.4 m, 4 spherical contact pads at (-0.10, +/-0.25, +/-0.15) m,
+    8 thruster mount sites at X=0.0 with the same corner layout. `base_link` is the sole root
+    link of this tree (no world/wall links here: the wall is MuJoCo-only geometry in
+    mjcf/rov_wall.xml and is rendered in RViz2 purely via the /rov/environment_markers topic).
+    All non-base links are rigidly fixed; the only real DOF is the floating base, which is
+    driven by AdhereMujocoHardware's free joint, not by any URDF joint.
   -->
   <material name="chassis_orange">
@@ -17,13 +19,4 @@
     <color rgba="0.6 0.6 0.6 1.0"/>
   </material>
-  <material name="wall_grey">
-    <color rgba="0.25 0.25 0.3 1.0"/>
-  </material>
-  <link name="world"/>
-  <joint name="world_to_base" type="fixed">
-    <parent link="world"/>
-    <child link="base_link"/>
-    <origin xyz="0.125 0 0.5" rpy="0 0 0"/>
-  </joint>
   <link name="base_link">
     <visual>
@@ -89,18 +82,3 @@
   <xacro:thruster_marker name="thr_T7" x="0.0" y="0.25" z="-0.15"/>
   <xacro:thruster_marker name="thr_T8" x="0.0" y="-0.25" z="-0.15"/>
-  <!-- Static wall plane, world X=0, outward normal +X, matching the MJCF's wall body at X=-0.01 -->
-  <link name="wall">
-    <visual>
-      <origin xyz="-0.01 0 0" rpy="0 0 0"/>
-      <geometry>
-        <box size="0.02 4.0 4.0"/>
-      </geometry>
-      <material name="wall_grey"/>
-    </visual>
-  </link>
-  <joint name="world_to_wall" type="fixed">
-    <parent link="world"/>
-    <child link="wall"/>
-    <origin xyz="0 0 0" rpy="0 0 0"/>
-  </joint>
 </robot>

File: src/descriptions/simplified_v1_description/xacro/ros2_control.xacro (robot description, xacro)
@@ -10,15 +10,13 @@
       - 8  pad_contact     (pad_*/force x4, pad_*/v_sep x4)
   -->
-  <xacro:arg name="wave_profile" default="calm"/>
   <xacro:arg name="headless" default="false"/>
   <ros2_control name="AdhereMujocoSystem" type="system">
     <hardware>
       <plugin>adhere_mujoco_hardware/AdhereMujocoHardware</plugin>
-      <param name="wave_profile">$(arg wave_profile)</param>
       <param name="headless">$(arg headless)</param>
     </hardware>
     <joint name="thr_N1">
       <command_interface name="effort">
-        <param name="min">22.0</param>
+        <param name="min">-40.0</param>
         <param name="max">40.0</param>
       </command_interface>
@@ -27,5 +25,5 @@
     <joint name="thr_N2">
       <command_interface name="effort">
-        <param name="min">22.0</param>
+        <param name="min">-40.0</param>
         <param name="max">40.0</param>
       </command_interface>
@@ -34,5 +32,5 @@
     <joint name="thr_N3">
       <command_interface name="effort">
-        <param name="min">22.0</param>
+        <param name="min">-40.0</param>
         <param name="max">40.0</param>
       </command_interface>
@@ -41,5 +39,5 @@
     <joint name="thr_N4">
       <command_interface name="effort">
-        <param name="min">22.0</param>
+        <param name="min">-40.0</param>
         <param name="max">40.0</param>
       </command_interface>
