Commit message: Phase 3.5: dual state-acquisition (ground_truth/sensor_fusion) + 6-DOF Xbox trigger teleop
Add a second, independent noisy multi-rate sensing path (500Hz IMU, 50Hz
Depth, 20Hz DVL, 500Hz load cells) alongside the existing noise-free ground
truth in AdhereMujocoHardware, fused by a new RovStateEstimator inside
AdhereController. Ground truth is now bound to private AdhereController
members (never CtrlInterfaces), and every FSMState reads exclusively from a
new CtrlInterfaces::ActiveState populated per estimation_mode -- enforcing
strict ground-truth isolation in sensor_fusion mode. Also complete Xbox
teleop to 6-DOF: LT/LB drives pitch_rate, RT/RB drives roll_rate, consumed by
StateOpenLoop (wrench) and StatePidHold (clamped tilt-angle setpoints).

Co-Authored-By: Claude Sonnet 5 <noreply@anthropic.com>

File: src/descriptions/simplified_v1_description/xacro/robot.xacro (robot description, xacro)
@@ -82,3 +82,30 @@
   <xacro:thruster_marker name="thr_T7" x="0.0" y="0.25" z="-0.15"/>
   <xacro:thruster_marker name="thr_T8" x="0.0" y="-0.25" z="-0.15"/>
+  <!-- Phase 3.5 sensor mounting markers (TF only, no physics): matches imu_site/depth_site/
+       dvl_site/loadcell_*_site positions in mjcf/rov_wall.xml exactly. -->
+  <material name="sensor_green">
+    <color rgba="0.2 1.0 0.2 1.0"/>
+  </material>
+  <xacro:macro name="sensor_marker" params="name x y z">
+    <link name="${name}">
+      <visual>
+        <geometry>
+          <sphere radius="0.015"/>
+        </geometry>
+        <material name="sensor_green"/>
+      </visual>
+    </link>
+    <joint name="base_to_${name}" type="fixed">
+      <parent link="base_link"/>
+      <child link="${name}"/>
+      <origin xyz="${x} ${y} ${z}" rpy="0 0 0"/>
+    </joint>
+  </xacro:macro>
+  <xacro:sensor_marker name="imu_link" x="0.0" y="0.0" z="0.0"/>
+  <xacro:sensor_marker name="depth_link" x="0.0" y="0.0" z="0.0"/>
+  <xacro:sensor_marker name="dvl_link" x="0.0" y="0.0" z="-0.20"/>
+  <xacro:sensor_marker name="loadcell_TL_link" x="-0.1" y="0.25" z="0.15"/>
+  <xacro:sensor_marker name="loadcell_TR_link" x="-0.1" y="-0.25" z="0.15"/>
+  <xacro:sensor_marker name="loadcell_BL_link" x="-0.1" y="0.25" z="-0.15"/>
+  <xacro:sensor_marker name="loadcell_BR_link" x="-0.1" y="-0.25" z="-0.15"/>
 </robot>

File: src/descriptions/simplified_v1_description/xacro/ros2_control.xacro (robot description, xacro)
@@ -3,10 +3,15 @@
   <!--
     ros2_control contract for AdhereMujocoHardware (ROS 2 Foxy hardware_interface::SystemInterface).
-    8 command_interface (thruster effort) + 36 state_interface, matching CLAUDE.md Sec.3/4 and
+    8 command_interface (thruster effort) + 55 state_interface, matching CLAUDE.md Sec.3/4 and
     this package's README interface table exactly:
       - 8  thruster effort readback
-      - 10 imu_sensor      (orientation.w/x/y/z, angular_velocity.x/y/z, linear_acceleration.x/y/z)
-      - 10 rov_odom        (pos.x/y/z, quat.w/x/y/z, vel_body.x/y/z)
-      - 8  pad_contact     (pad_*/force x4, pad_*/v_sep x4)
+      - 10 imu_sensor      (orientation.w/x/y/z, angular_velocity.x/y/z, linear_acceleration.x/y/z), ground truth
+      - 10 rov_odom        (pos.x/y/z, quat.w/x/y/z, vel_body.x/y/z), ground truth
+      - 8  pad_contact     (pad_*/force x4, pad_*/v_sep x4), ground truth
+      - 10 imu_sensor_noisy    (same layout as imu_sensor, 500Hz noisy IMU)
+      - 1  depth_sensor_noisy (z, 50Hz sample-and-hold noisy depth)
+      - 4  dvl_sensor_noisy   (vel.x/y/z + range, 20Hz sample-and-hold noisy DVL)
+      - 4  loadcell_noisy     (pad_*/force x4, 500Hz noisy load cells)
+    (Phase 3.5, CLAUDE.md dual state-acquisition: ground_truth vs sensor_fusion.)
   -->
   <ros2_control name="AdhereMujocoSystem" type="system">
@@ -104,4 +109,33 @@
       <state_interface name="pad_BR/v_sep"/>
     </sensor>
+    <!-- Phase 3.5 realistic noisy multi-rate sensors: a second, independent sensing path from
+         the 3 ground-truth sensors above, consumed only by RovStateEstimator. -->
+    <sensor name="imu_sensor_noisy">
+      <state_interface name="orientation.w"/>
+      <state_interface name="orientation.x"/>
+      <state_interface name="orientation.y"/>
+      <state_interface name="orientation.z"/>
+      <state_interface name="angular_velocity.x"/>
+      <state_interface name="angular_velocity.y"/>
+      <state_interface name="angular_velocity.z"/>
+      <state_interface name="linear_acceleration.x"/>
+      <state_interface name="linear_acceleration.y"/>
+      <state_interface name="linear_acceleration.z"/>
+    </sensor>
+    <sensor name="depth_sensor_noisy">
+      <state_interface name="z"/>
+    </sensor>
+    <sensor name="dvl_sensor_noisy">
+      <state_interface name="vel.x"/>
+      <state_interface name="vel.y"/>
+      <state_interface name="vel.z"/>
+      <state_interface name="range"/>
+    </sensor>
+    <sensor name="loadcell_noisy">
+      <state_interface name="pad_TL/force"/>
+      <state_interface name="pad_TR/force"/>
+      <state_interface name="pad_BL/force"/>
+      <state_interface name="pad_BR/force"/>
+    </sensor>
   </ros2_control>
 </robot>
